File: hardware/leveling_package.kicad_pcb (KiCad board)
At the start: 2 copper layers, 74 x 74 mm, 3 parts, among them J1 Conn_01x16_Male, J2 Conn_01x16_Male

Commit message: 2nd leg
Other:
- board size 74 x 74 mm -> 100 x 74 mm
Changed lines of the file:
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@@
   (general
     (thickness 1.6)
-    (drawings 10)
+    (drawings 16)
     (tracks 0)
     (zones 0)
@@
     )
   )
+  (gr_line (start 31.07107 24) (end 57.07107 50) (layer Edge.Cuts) (width 0.05))
+  (gr_line (start 24 31.07107) (end 31.07107 24) (layer Edge.Cuts) (width 0.05))
+  (gr_line (start 50 57.07107) (end 24 31.07107) (layer Edge.Cuts) (width 0.05))
+  (gr_line (start 24 31.07107) (end 74 81.07107) (layer F.SilkS) (width 0.12))
+  (gr_line (start 31.07107 24) (end 74 66.92893) (layer F.SilkS) (width 0.12))
+  (gr_line (start 24 24) (end 74 74) (layer F.SilkS) (width 0.12))
   (gr_line (start 116.92893 24) (end 124 31.07107) (layer Edge.Cuts) (width 0.05))
   (gr_line (start 124 31.07107) (end 98 57.07107) (layer Edge.Cuts) (width 0.05))
@@
   (gr_line (start 50 98) (end 98 98) (layer Edge.Cuts) (width 0.05))
   (gr_line (start 98 57.07107) (end 98 98) (layer Edge.Cuts) (width 0.05))
-  (gr_line (start 50 50) (end 50 98) (layer Edge.Cuts) (width 0.05))
-  (gr_line (start 50 50) (end 90.92893 50) (layer Edge.Cuts) (width 0.05))
+  (gr_line (start 50 57.07107) (end 50 98) (layer Edge.Cuts) (width 0.05))
+  (gr_line (start 57.07107 50) (end 90.92893 50) (layer Edge.Cuts) (width 0.05))
 )

Commit message: 3rd leg
Other:
- board size 100 x 74 mm -> 100 x 100 mm
Changed lines of the file:
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@@
   (general
     (thickness 1.6)
-    (drawings 16)
+    (drawings 22)
     (tracks 0)
     (zones 0)
@@
     )
   )
+  (gr_line (start 24 116.92893) (end 31.07107 124) (layer Edge.Cuts) (width 0.05))
+  (gr_line (start 31.07107 124) (end 57.07107 98) (layer Edge.Cuts) (width 0.05))
+  (gr_line (start 50 90.92893) (end 24 116.92893) (layer Edge.Cuts) (width 0.05))
+  (gr_line (start 31.07107 124) (end 74 81.07107) (layer F.SilkS) (width 0.12))
+  (gr_line (start 24 116.92893) (end 74 66.92893) (layer F.SilkS) (width 0.12))
+  (gr_line (start 24 124) (end 74 74) (layer F.SilkS) (width 0.12))
   (gr_line (start 31.07107 24) (end 57.07107 50) (layer Edge.Cuts) (width 0.05))
   (gr_line (start 24 31.07107) (end 31.07107 24) (layer Edge.Cuts) (width 0.05))
@@
   (gr_line (start 74 81.07107) (end 124 31.07107) (layer F.SilkS) (width 0.12))
   (gr_line (start 74 74) (end 124 24) (layer F.SilkS) (width 0.12))
-  (gr_line (start 50 98) (end 98 98) (layer Edge.Cuts) (width 0.05))
+  (gr_line (start 57.07107 98) (end 98 98) (layer Edge.Cuts) (width 0.05))
   (gr_line (start 98 57.07107) (end 98 98) (layer Edge.Cuts) (width 0.05))
-  (gr_line (start 50 57.07107) (end 50 98) (layer Edge.Cuts) (width 0.05))
+  (gr_line (start 50 57.07107) (end 50 90.92893) (layer Edge.Cuts) (width 0.05))
   (gr_line (start 57.07107 50) (end 90.92893 50) (layer Edge.Cuts) (width 0.05))
 )
